Commit message: modified some path problems

File: src/perception_pipeline/urdf/realsense_d435/camera.urdf.xacro (robot description, xacro)
@@ -34,5 +34,5 @@
             <origin xyz="${d435_cam_mount_from_center_offset} ${-d435_cam_depth_py} 0" rpy="${pi/2} 0 ${pi/2}"/>
             <geometry>
-                <mesh filename="$(find moveit2_tutorials)/meshes/d435.dae" />
+                <mesh filename="$(find perception_pipeline)/meshes/d435.dae" />
             </geometry>
         </visual>
